File: HW2/PIC32 PCB/PIC32Circuit.sch (EAGLE design)
At the start: 22 parts, among them J1 USB-MB-H

Commit message: Board Updates
Parts:
- removed C1*, C1*1: (no value), PIC32:CPOL-USCT3216
- added C5, C6: 10uF, resistor:CPOL-USTT2D4
- C1, C2: value (none) -> 1uF
- C3: value (none) -> .1uF
- C4: value (none) -> 0.1uF
- R1, R2: value (none) -> 10k
- R4, R5: value (none) -> 330
- RES: value (none) -> 8MHz
- renumbered PBSWITCH to PBS2, PBSWITCH1 to PBS1, RESONATOR to RES
Connections:
- net 3V3: now also C5.+; no longer C1*.+
- net GND: now also C5.-, C6.-; no longer C1*.-, C1*1.-
- net N$3: now also C6.+; no longer C1*1.+
Changed lines of the file:
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@@
 </classes>
 <parts>
-<part name="R4" library="resistor" deviceset="R-US_" device="0207/10"/>
+<part name="R4" library="resistor" deviceset="R-US_" device="0207/10" value="330"/>
 <part name="LED1" library="led" deviceset="LED" device="3MM"/>
-<part name="C1" library="PIC32" deviceset="C-US" device="025-024X044"/>
-<part name="C1*" library="PIC32" deviceset="CPOL-US" device="CT3216"/>
+<part name="C1" library="PIC32" deviceset="C-US" device="025-024X044" value="1uF"/>
 <part name="U$1" library="PIC32" deviceset="PIC32MX250F128B" device=""/>
 <part name="U$2" library="PIC32" deviceset="SLIDERSWITCH" device=""/>
 <part name="J1" library="PIC32" deviceset="USB" device="-MB-H"/>
-<part name="RESONATOR" library="PIC32" deviceset="M03" device="PTH"/>
+<part name="RES" library="PIC32" deviceset="M03" device="PTH" value="8MHz"/>
 <part name="J4" library="PIC32" deviceset="M08" device=""/>
 <part name="J5" library="PIC32" deviceset="M08" device=""/>
 <part name="U$3" library="PIC32" deviceset="MCP1702" device=""/>
 <part name="PICKIT3" library="PIC32" deviceset="M06" device="SILK_FEMALE_PTH"/>
-<part name="C2" library="PIC32" deviceset="C-US" device="025-024X044"/>
-<part name="C3" library="PIC32" deviceset="C-US" device="025-024X044"/>
-<part name="C4" library="PIC32" deviceset="C-US" device="025-024X044"/>
-<part name="PBSWITCH" library="PIC32" deviceset="M03" device="PTH"/>
-<part name="R1" library="resistor" deviceset="R-US_" device="0207/10"/>
-<part name="R2" library="resistor" deviceset="R-US_" device="0207/10"/>
-<part name="PBSWITCH1" library="PIC32" deviceset="M03" device="PTH"/>
-<part name="R5" library="resistor" deviceset="R-US_" device="0207/10"/>
+<part name="C2" library="PIC32" deviceset="C-US" device="025-024X044" value="1uF"/>
+<part name="C3" library="PIC32" deviceset="C-US" device="025-024X044" value=".1uF"/>
+<part name="C4" library="PIC32" deviceset="C-US" device="025-024X044" value="0.1uF"/>
+<part name="PBS2" library="PIC32" deviceset="M03" device="PTH"/>
+<part name="R1" library="resistor" deviceset="R-US_" device="0207/10" value="10k"/>
+<part name="R2" library="resistor" deviceset="R-US_" device="0207/10" value="10k"/>
+<part name="PBS1" library="PIC32" deviceset="M03" device="PTH"/>
+<part name="R5" library="resistor" deviceset="R-US_" device="0207/10" value="330"/>
 <part name="LED3" library="led" deviceset="LED" device="3MM"/>
-<part name="C1*1" library="PIC32" deviceset="CPOL-US" device="CT3216"/>
+<part name="C5" library="resistor" deviceset="CPOL-US" device="TT2D4" value="10uF"/>
+<part name="C6" library="resistor" deviceset="CPOL-US" device="TT2D4" value="10uF"/>
 </parts>
 <sheets>
@@
 <instance part="LED1" gate="G$1" x="152.4" y="205.74" rot="R90"/>
 <instance part="C1" gate="G$1" x="73.66" y="200.66"/>
-<instance part="C1*" gate="G$1" x="185.42" y="210.82" rot="R180"/>
 <instance part="U$1" gate="G$1" x="111.76" y="152.4"/>
 <instance part="U$2" gate="G$1" x="88.9" y="213.36" rot="R90"/>
 <instance part="J1" gate="G$1" x="114.3" y="215.9" rot="R90"/>
-<instance part="RESONATOR" gate="J$1" x="43.18" y="134.62"/>
+<instance part="RES" gate="J$1" x="43.18" y="134.62"/>
 <instance part="J4" gate="G$1" x="180.34" y="127" rot="R180"/>
 <instance part="J5" gate="G$1" x="182.88" y="175.26" rot="R180"/>
@@
 <instance part="C3" gate="G$1" x="139.7" y="182.88"/>
 <instance part="C4" gate="G$1" x="78.74" y="134.62"/>
-<instance part="PBSWITCH" gate="J$1" x="40.64" y="172.72" rot="R270"/>
+<instance part="PBS2" gate="J$1" x="40.64" y="172.72" rot="R270"/>
 <instance part="R1" gate="G$1" x="53.34" y="152.4"/>
 <instance part="R2" gate="G$1" x="40.64" y="96.52"/>
-<instance part="PBSWITCH1" gate="J$1" x="50.8" y="86.36" rot="R180"/>
+<instance part="PBS1" gate="J$1" x="50.8" y="86.36" rot="R180"/>
 <instance part="R5" gate="G$1" x="40.64" y="114.3"/>
 <instance part="LED3" gate="G$1" x="53.34" y="114.3" rot="R90"/>
-<instance part="C1*1" gate="G$1" x="144.78" y="142.24" rot="R90"/>
+<instance part="C5" gate="G$1" x="185.42" y="210.82" rot="R180"/>
+<instance part="C6" gate="G$1" x="144.78" y="142.24" rot="R90"/>
 </instances>
 <busses>
 </busses>
 <nets>
-<net name="N$1" class="0">
-<segment>
-<wire x1="121.92" y1="104.14" x2="121.92" y2="106.68" width="0.1524" layer="91"/>
-</segment>
-</net>
 <net name="GND" class="0">
 <segment>
@@
 </segment>
 <segment>
-<pinref part="C1*" gate="G$1" pin="-"/>
 <wire x1="185.42" y1="215.9" x2="185.42" y2="218.44" width="0.1524" layer="91"/>
 <label x="185.42" y="220.98" size="1.778" layer="95"/>
+<pinref part="C5" gate="G$1" pin="-"/>
 </segment>
 <segment>
@@
 </segment>
 <segment>
-<pinref part="RESONATOR" gate="J$1" pin="2"/>
+<pinref part="RES" gate="J$1" pin="2"/>
 <wire x1="50.8" y1="134.62" x2="55.88" y2="134.62" width="0.1524" layer="91"/>
 <label x="58.42" y="134.62" size="1.778" layer="95"/>
@@
 </segment>
 <segment>
-<pinref part="PBSWITCH" gate="J$1" pin="1"/>
+<pinref part="PBS2" gate="J$1" pin="1"/>
 <wire x1="38.1" y1="165.1" x2="38.1" y2="157.48" width="0.1524" layer="91"/>
 <wire x1="38.1" y1="157.48" x2="33.02" y2="157.48" width="0.1524" layer="91"/>
@@
 </segment>
 <segment>
-<pinref part="PBSWITCH1" gate="J$1" pin="3"/>
+<pinref part="PBS1" gate="J$1" pin="3"/>
 <wire x1="43.18" y1="83.82" x2="33.02" y2="83.82" width="0.1524" layer="91"/>
 <label x="27.94" y="83.82" size="1.778" layer="95"/>
@@
 </segment>
 <segment>
-<pinref part="C1*1" gate="G$1" pin="-"/>
 <wire x1="149.86" y1="142.24" x2="152.4" y2="142.24" width="0.1524" layer="91"/>
 <label x="152.4" y="142.24" size="1.778" layer="95"/>
+<pinref part="C6" gate="G$1" pin="-"/>
 </segment>
 <segment>
@@
 <junction x="175.26" y="200.66"/>
 <wire x1="185.42" y1="200.66" x2="185.42" y2="208.28" width="0.1524" layer="91"/>
-<pinref part="C1*" gate="G$1" pin="+"/>
+<pinref part="C5" gate="G$1" pin="+"/>
 </segment>
 <segment>
@@
 <net name="OSC2" class="0">
 <segment>
-<pinref part="RESONATOR" gate="J$1" pin="3"/>
+<pinref part="RES" gate="J$1" pin="3"/>
 <wire x1="50.8" y1="137.16" x2="55.88" y2="137.16" width="0.1524" layer="91"/>
 <label x="55.88" y="139.7" size="1.778" layer="95"/>
@@
 <net name="OSC1" class="0">
 <segment>
-<pinref part="RESONATOR" gate="J$1" pin="1"/>
+<pinref part="RES" gate="J$1" pin="1"/>
 <wire x1="50.8" y1="132.08" x2="55.88" y2="132.08" width="0.1524" layer="91"/>
 <label x="55.88" y="129.54" size="1.778" layer="95"/>
@@
 <junction x="66.04" y="157.48"/>
 <wire x1="66.04" y1="157.48" x2="43.18" y2="157.48" width="0.1524" layer="91"/>
-<pinref part="PBSWITCH" gate="J$1" pin="3"/>
+<pinref part="PBS2" gate="J$1" pin="3"/>
 <wire x1="43.18" y1="157.48" x2="43.18" y2="165.1" width="0.1524" layer="91"/>
 <pinref part="R1" gate="G$1" pin="2"/>
@@
 <wire x1="33.02" y1="88.9" x2="43.18" y2="88.9" width="0.1524" layer="91"/>
 <label x="25.4" y="96.52" size="1.778" layer="95"/>
-<pinref part="PBSWITCH1" gate="J$1" pin="1"/>
+<pinref part="PBS1" gate="J$1" pin="1"/>
 </segment>
 <segment>
@@
 <segment>
 <pinref part="U$1" gate="G$1" pin="20.VCAP"/>
-<pinref part="C1*1" gate="G$1" pin="+"/>
 <wire x1="127" y1="142.24" x2="142.24" y2="142.24" width="0.1524" layer="91"/>
+<pinref part="C6" gate="G$1" pin="+"/>
 </segment>
 </net>
@@
 </sheet>
 </sheets>
+<errors>
+</errors>
 </schematic>
 </drawing>
